File: STM32/STM32.kicad_pcb (KiCad board)
At the start: 2 copper layers, 83.1 x 37.2 mm, 63 parts, among them J1 USB_C_Receptacle_USB2.0, J2 Conn_01x02, J3 Conn_01x04, J4 Conn_01x19, J5 Conn_01x20, J6 Conn_01x02, J7 Conn_01x03, Q1 Si2301, SW1 SW_Push, SW2 SW_Push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

Commit message: PCB更新
Routing:
- net +3V3: track 286.4 -> 287.1 mm
- net GND: vias 41 -> 43

Commit message: PCB更新
Other:
- board text added: "+3V3"
- board text added: "3V3_DEBUG"
- board text added: "A1"
- board text added: "B1"
- board text added: "BOOT0"
- board text added: "GND"
- board text added: "PA0"
- board text added: "PA1"
- board text added: "PA10"
- board text added: "PA11"
- board text added: "PA12"
- board text added: "PA15"
- board text added: "PA2"
- board text added: "PA3"
- board text added: "PA4"
- board text added: "PA5"
- board text added: "PA6"
- board text added: "PA7"
- board text added: "PA8"
- board text added: "PA9"
- board text added: "PB0"
- board text added: "PB1"
- board text added: "PB10"
- board text added: "PB11"
- board text added: "PB12"
- board text added: "PB13"
- board text added: "PB14"
- board text added: "PB15"
- board text added: "PB2"
- board text added: "PB3"
- board text added: "PB4"
- board text added: "PB5"
- board text added: "PB6"
- board text added: "PB7"
- board text added: "PB8"
- board text added: "PB9"
- board text added: "PC14"
- board text added: "PC15"
- board text added: "SWCLK"
- board text added: "SWDIO"
- board text added: "VBUS"
- board text added: "W1"
Changed lines of the file:
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@@
     (property "Sheetname" "STM32_MinimumSystem")
     (attr smd)
-    (fp_text reference "Y1" (at 0 -2.45 90) (layer "F.SilkS")
+    (fp_text reference "Y1" (at 4 0.09 90) (layer "F.SilkS")
       (effects (font (size 1 1) (thickness 0.15)))
     )
@@
   (gr_line (start 39.2 95.8) (end 39.2 97.2) (layer "Margin") (width 0.15))
   (gr_line (start 39.2 98.4) (end 39.2 99.8) (layer "Margin") (width 0.15))
+  (gr_text "W1" (at 90.88 92.46) (layer "F.SilkS")
+    (effects (font (size 0.6 0.6) (thickness 0.1)))
+  )
+  (gr_text "BOOT0" (at 81.91 115.33) (layer "F.SilkS")
+    (effects (font (size 0.6 0.6) (thickness 0.1)))
+  )
+  (gr_text "+3V3" (at 59.35 111.5) (layer "F.SilkS")
+    (effects (font (size 0.6 0.6) (thickness 0.1)))
+  )
+  (gr_text "PA9\n" (at 43.87 115.29) (layer "F.SilkS")
+    (effects (font (size 0.6 0.6) (thickness 0.1)))
+  )
+  (gr_text "PB10" (at 58.98 94) (layer "F.SilkS")
+    (effects (font (size 1 0.6) (thickness 0.15)))
+  )
+  (gr_text "PA4" (at 76.63 93.91) (layer "F.SilkS")
+    (effects (font (size 1 0.6) (thickness 0.15)))
+  )
+  (gr_text "BOOT0" (at 62.19 111.55) (layer "F.SilkS")
+    (effects (font (size 0.6 0.6) (thickness 0.1)))
+  )
+  (gr_text "PA5" (at 74.22 93.9) (layer "F.SilkS")
+    (effects (font (size 1 0.6) (thickness 0.15)))
+  )
+  (gr_text "SWDIO" (at 87.63 107.54) (layer "F.SilkS")
+    (effects (font (size 1 0.6) (thickness 0.15)))
+  )
+  (gr_text "VBUS\n" (at 43.63 93.94) (layer "F.SilkS")
+    (effects (font (size 1 0.6) (thickness 0.15)))
+  )
+  (gr_text "GND" (at 41.15 93.94) (layer "F.SilkS")
+    (effects (font (size 1 0.6) (thickness 0.15)))
+  )
+  (gr_text "+3V3" (at 84.45 115.32) (layer "F.SilkS")
+    (effects (font (size 0.6 0.6) (thickness 0.1)))
+  )
+  (gr_text "PC15" (at 79.35 115.33) (layer "F.SilkS")
+    (effects (font (size 0.6 0.6) (thickness 0.1)))
+  )
+  (gr_text "PA10" (at 46.47 115.31) (layer "F.SilkS")
+    (effects (font (size 0.6 0.6) (thickness 0.1)))
+  )
+  (gr_text "PB5" (at 61.56 115.4) (layer "F.SilkS")
+    (effects (font (size 0.6 0.6) (thickness 0.1)))
+  )
+  (gr_text "PB4" (at 59 115.4) (layer "F.SilkS")
+    (effects (font (size 0.6 0.6) (thickness 0.1)))
+  )
+  (gr_text "PA3" (at 79.19 93.95) (layer "F.SilkS")
+    (effects (font (size 1 0.6) (thickness 0.15)))
+  )
+  (gr_text "PA7" (at 69.18 93.89) (layer "F.SilkS")
+    (effects (font (size 1 0.6) (thickness 0.15)))
+  )
+  (gr_text "PB9" (at 71.67 115.31) (layer "F.SilkS")
+    (effects (font (size 0.6 0.6) (thickness 0.1)))
+  )
+  (gr_text "GND\n" (at 88.56 112.78) (layer "F.SilkS")
+    (effects (font (size 1 0.6) (thickness 0.15)))
+  )
+  (gr_text "SWCLK\n" (at 87.58 109.88) (layer "F.SilkS")
+    (effects (font (size 1 0.6) (thickness 0.15)))
+  )
+  (gr_text "PA11" (at 48.91 115.34) (layer "F.SilkS")
+    (effects (font (size 0.6 0.6) (thickness 0.1)))
+  )
+  (gr_text "PA0" (at 86.92 93.9) (layer "F.SilkS")
+    (effects (font (size 1 0.6) (thickness 0.15)))
+  )
+  (gr_text "PA15\n" (at 53.9 115.31) (layer "F.SilkS")
+    (effects (font (size 0.6 0.6) (thickness 0.1)))
+  )
+  (gr_text "PB1" (at 64.05 93.95) (layer "F.SilkS")
+    (effects (font (size 1 0.6) (thickness 0.15)))
+  )
+  (gr_text "PA8" (at 41.1 115.22) (layer "F.SilkS")
+    (effects (font (size 0.6 0.6) (thickness 0.1)))
+  )
+  (gr_text "PB8" (at 69.04 115.31) (layer "F.SilkS")
+    (effects (font (size 0.6 0.6) (thickness 0.1)))
+  )
+  (gr_text "PB0" (at 66.59 93.94) (layer "F.SilkS")
+    (effects (font (size 1 0.6) (thickness 0.15)))
+  )
+  (gr_text "PB10" (at 74.28 115.37) (layer "F.SilkS")
+    (effects (font (size 0.6 0.6) (thickness 0.1)))
+  )
+  (gr_text "PB14" (at 48.75 93.95) (layer "F.SilkS")
+    (effects (font (size 1 0.6) (thickness 0.15)))
+  )
+  (gr_text "PB13" (at 51.4 93.91) (layer "F.SilkS")
+    (effects (font (size 1 0.6) (thickness 0.15)))
+  )
+  (gr_text "PB12" (at 53.92 93.97) (layer "F.SilkS")
+    (effects (font (size 1 0.6) (thickness 0.15)))
+  )
+  (gr_text "PA1" (at 84.34 93.9) (layer "F.SilkS")
+    (effects (font (size 1 0.6) (thickness 0.15)))
+  )
+  (gr_text "PB6\n" (at 64.2 115.31) (layer "F.SilkS")
+    (effects (font (size 0.6 0.6) (thickness 0.1)))
+  )
+  (gr_text "PB2\n" (at 61.58 93.98) (layer "F.SilkS")
+    (effects (font (size 1 0.6) (thickness 0.15)))
+  )
+  (gr_text "PA2" (at 81.77 93.91) (layer "F.SilkS")
+    (effects (font (size 1 0.6) (thickness 0.15)))
+  )
+  (gr_text "+3V3" (at 87.06 115.32) (layer "F.SilkS")
+    (effects (font (size 0.6 0.6) (thickness 0.1)))
+  )
+  (gr_text "PB7\n" (at 66.58 115.35) (layer "F.SilkS")
+    (effects (font (size 0.6 0.6) (thickness 0.1)))
+  )
+  (gr_text "A1" (at 90.86 91.28) (layer "F.SilkS")
+    (effects (font (size 0.6 0.6) (thickness 0.1)))
+  )
+  (gr_text "GND" (at 89.59 115.33) (layer "F.SilkS")
+    (effects (font (size 0.6 0.6) (thickness 0.1)))
+  )
+  (gr_text "PC14" (at 76.85 115.36) (layer "F.SilkS")
+    (effects (font (size 0.6 0.6) (thickness 0.1)))
+  )
+  (gr_text "PB3" (at 56.47 115.31) (layer "F.SilkS")
+    (effects (font (size 0.6 0.6) (thickness 0.1)))
+  )
+  (gr_text "B1\n" (at 90.86 93.53) (layer "F.SilkS")
+    (effects (font (size 0.6 0.6) (thickness 0.1)))
+  )
+  (gr_text "PB11" (at 56.44 93.99) (layer "F.SilkS")
+    (effects (font (size 1 0.6) (thickness 0.15)))
+  )
+  (gr_text "PA6" (at 71.71 93.86) (layer "F.SilkS")
+    (effects (font (size 1 0.6) (thickness 0.15)))
+  )
+  (gr_text "3V3_DEBUG\n" (at 86.89 105.02) (layer "F.SilkS")
+    (effects (font (size 1 0.6) (thickness 0.15)))
+  )
+  (gr_text "PA12" (at 51.51 115.32) (layer "F.SilkS")
+    (effects (font (size 0.6 0.6) (thickness 0.1)))
+  )
+  (gr_text "PB15\n" (at 46.26 93.97) (layer "F.SilkS")
+    (effects (font (size 1 0.6) (thickness 0.15)))
+  )
   (segment (start 53.05 104) (end 59.8 104) (width 0.381) (layer "F.Cu") (net 1))
   (segment (start 81.075 123.25) (end 79.075 125.25) (width 0.381) (layer "F.Cu") (net 1))
